Commit message: feat: add localization, inspection, and experiment results

File: robot_data/urdf/robot.urdf (robot description, URDF)
Before this commit: robot robot_xj, 4 links, 3 joints
Joints:
- joint imu_joint: origin xyz=0.40 0.30 0.15 rpy=0 0 0.78539816340 -> xyz=0.37 0.28 0.15 rpy=0 0 0.8229227423153264
